Commit message: Add mass to the robot's links.
The masses come from https://github.com/iit-DLSLab/hyq-description/blob/master/urdfs/common.xacro

This solves the nan jacobians pinocchio problem.

File: examples/hyq/hyq_urdf/urdf/hyq.urdf (robot description, URDF)
Before this commit: robot hyq, 18 links, 17 joints
Links:
- link lf_hipassembly: mass None -> 2.93
- link lf_lowerleg: mass None -> 0.811
- link lf_upperleg: mass None -> 2.638
- link lh_hipassembly: mass None -> 2.93
- link lh_lowerleg: mass None -> 0.811
- link lh_upperleg: mass None -> 2.638
- link rf_hipassembly: mass None -> 2.93
- link rf_lowerleg: mass None -> 0.811
- link rf_upperleg: mass None -> 2.638
- link rh_hipassembly: mass None -> 2.93
- link rh_lowerleg: mass None -> 0.811
- link rh_upperleg: mass None -> 2.638
- link trunk: mass None -> 58.96
